File: KiCAD/Z80-GRANT.sch (KiCad schematic (older format))
At the start: 39 parts, among them J1 ACIA-J, J2 Conn_01x06, J3 SBC8080 BUS, J4 Jack-DC, M1 MountingHole_M3, M2 MountingHole_M3, M3 MountingHole_M3, M4 MountingHole_M3, SW1 SW_Push, SW2 SW_SPDT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

Commit message: 回路図イメージ、部品表追加
Parts:
- RN1: value R_Network08 -> 10k
- U5: value 74LS138 -> 74HC138
- U7: value 74LS32 -> 74HC32
Changed lines of the file:
@@
 encoding utf-8
 Sheet 1 1
-Title "Z80 Sigleboard Computer"
-Date "2018/9/8"
+Title "Z80 Sigleboard Computer (w/MC6850)"
+Date "2018-12-28"
 Rev "1"
 Comp ""
@@
 P 7100 4450
 F 0 "U7" H 7100 4500 50  0000 C CNN
-F 1 "74LS32" H 7100 4400 50  0000 C CNN
+F 1 "74HC32" H 7100 4400 50  0000 C CNN
 F 2 "Housings_DIP:DIP-14_W7.62mm_Socket" H 7100 4450 50  0001 C CNN
 F 3 "" H 7100 4450 50  0001 C CNN
@@
 P 7100 5000
 F 0 "U7" H 7100 5050 50  0000 C CNN
-F 1 "74LS32" H 7100 4950 50  0000 C CNN
+F 1 "74HC32" H 7100 4950 50  0000 C CNN
 F 2 "Housings_DIP:DIP-14_W7.62mm_Socket" H 7100 5000 50  0001 C CNN
 F 3 "" H 7100 5000 50  0001 C CNN
@@
 P 7100 5550
 F 0 "U7" H 7100 5600 50  0000 C CNN
-F 1 "74LS32" H 7100 5500 50  0000 C CNN
+F 1 "74HC32" H 7100 5500 50  0000 C CNN
 F 2 "Housings_DIP:DIP-14_W7.62mm_Socket" H 7100 5550 50  0001 C CNN
 F 3 "" H 7100 5550 50  0001 C CNN
@@
 P 7100 6100
 F 0 "U7" H 7100 6150 50  0000 C CNN
-F 1 "74LS32" H 7100 6050 50  0000 C CNN
+F 1 "74HC32" H 7100 6050 50  0000 C CNN
 F 2 "Housings_DIP:DIP-14_W7.62mm_Socket" H 7100 6100 50  0001 C CNN
 F 3 "" H 7100 6100 50  0001 C CNN
@@
 P 4350 3800
 F 0 "U5" H 4450 4300 50  0000 C CNN
-F 1 "74LS138" H 4500 3251 50  0000 C CNN
+F 1 "74HC138" H 4500 3251 50  0000 C CNN
 F 2 "Housings_DIP:DIP-16_W7.62mm_Socket" H 4350 3800 50  0001 C CNN
 F 3 "" H 4350 3800 50  0001 C CNN
@@
 P 2600 950
 F 0 "RN1" V 2100 950 50  0000 C CNN
-F 1 "R_Network08" V 3000 950 50  0000 C CNN
+F 1 "10k" V 3000 950 50  0000 C CNN
 F 2 "Resistors_THT:R_Array_SIP9" V 3075 950 50  0001 C CNN
 F 3 "" H 2600 950 50  0001 C CNN
